Commit message: feat:为各个组件增加了collision碰撞属性

File: chapt6/chapt6_ws/src/fishbot_description/urdf/fishbot/actuator/caster.urdf.xacro (robot description, xacro)
@@ -12,4 +12,13 @@
 				</material>
 			</visual>
+			<collision>
+				<origin xyz="0 0 0" rpy="0 0 0" />
+				<geometry>
+					<sphere radius="0.016" />
+				</geometry>
+				<material name="yellow">
+					<color rgba="1.0 1.0 0.0 0.8" />
+				</material>
+			</collision>
 		</link>
 		<joint name="${caster_name}_caster_joint" type="fixed">

File: chapt6/chapt6_ws/src/fishbot_description/urdf/fishbot/actuator/wheel.urdf.xacro (robot description, xacro)
@@ -12,4 +12,13 @@
 				</material>
 			</visual>
+			<collision>
+				<origin xyz="0 0 0" rpy="1.57079 0 0" />
+				<geometry>
+					<cylinder length="0.04" radius="0.032" />
+				</geometry>
+				<material name="yellow">
+					<color rgba="1.0 1.0 0.0 0.8" />
+				</material>
+			</collision>
 		</link>
 		<joint name="${wheel_name}_wheel_joint" type="continuous">

File: chapt6/chapt6_ws/src/fishbot_description/urdf/fishbot/base.urdf.xacro (robot description, xacro)
@@ -18,4 +18,13 @@
 				</material>
 			</visual>
+			<collision>
+				<origin xyz="0 0 0.0" rpy="0 0 0 " />
+				<geometry>
+					<cylinder length="${length}" radius="${radius}" />
+				</geometry>
+				<material name="white">
+					<color rgba="1.0 1.0 1.0 0.5"/>
+				</material>
+			</collision>
 		</link>
 	</xacro:macro>

File: chapt6/chapt6_ws/src/fishbot_description/urdf/fishbot/sensor/camera.urdf.xacro (robot description, xacro)
@@ -13,4 +13,13 @@
 				</material>
 			</visual>
+			<collision>
+				<origin xyz="0 0 0.0" rpy="0 0 0" />
+				<geometry>
+					<box size="0.02 0.10 0.02" />
+				</geometry>
+				<material name="green">
+					<color rgba="0.0 1.0 0.0 0.8"/>
+				</material>
+			</collision>
 		</link>
 		<joint name="camera_joint" type="fixed">

File: chapt6/chapt6_ws/src/fishbot_description/urdf/fishbot/sensor/imu.urdf.xacro (robot description, xacro)
@@ -12,4 +12,13 @@
 				</material>
 			</visual>
+			<collision>
+				<origin xyz="0 0 00" rpy="0 0 0 " />
+				<geometry>
+					<box size="0.02 0.02 0.02" />
+				</geometry>
+				<material name="black">
+					<color rgba = "0 0 0 0.8" />
+				</material>
+			</collision>
 		</link>
 		<joint name="imu_joint" type="fixed">

File: chapt6/chapt6_ws/src/fishbot_description/urdf/fishbot/sensor/laser.urdf.xacro (robot description, xacro)
@@ -13,4 +13,13 @@
 				</material>
 			</visual>
+			<collision>
+				<origin xyz="0 0 0" rpy="0 0 0" />
+				<geometry>
+					<cylinder length="0.10" radius="0.01" />
+				</geometry>
+				<material name="red">
+					<color rgba="0.0 1.0 0.0 0.8" />
+				</material>
+			</collision>
 		</link>
 		<joint name="laser_cylinder_joint" type="fixed">
@@ -30,4 +39,13 @@
 				</material>
 			</visual>
+			<collision>
+				<origin xyz="0 0 0" rpy="0 0 0 " />
+				<geometry>
+					<cylinder length="0.02" radius="0.02" />
+				</geometry>
+				<material name="green">
+					<color rgba="0.0 1.0 0.0 0.8" />
+				</material>
+			</collision>
 		</link>
 		<!-- 下面整段的意思是，将laser_link放到laser_cylinder_link 的上方0.05米的位置 -->
